File: hardware/lte-power-switch/lte-power-switch.kicad_pcb (KiCad board)
At the start: 2 copper layers, 38 x 28 mm, 15 parts, among them J1 HY2.0-4P-WT, J2 HY2.0-4P-WT, J3 HY2.0-4P-WT, U1 TPS22918DBVR

Commit message: feat(#88): ロードスイッチ基板 rev B（Grove コネクタの鏡像を修正）
rev A は、HY2.0-4P-WT のフットプリントの pad 番号が実物と鏡像だった
（三角のパッドに、Grove ケーブルの黒（GND）が来る）。rev B で直す。

- フットプリントの pad 番号を逆にした（1↔4、2↔3）。回路図（論理）は変えない
- コネクタまわりの配線を引き直した。SIG1・SIG2 は裏面の入れ子の U 字。
  U1・C1・C2・R1・R2・C3 と J1〜J3 の位置・向きは rev A と同じ（CPL も同じ）。
  TP2 のみ、VLTE の線の上に移した。テストポイントは rev A のまま
- 印字: 各コネクタに「tri=GND(black)」、裏面に全ピンの対応表。rev B #88
- scripts/check_gerber_connectivity.py を追加: 製造用ガーバーから銅箔の接続を求め、
  ネットの断線・ショート、J1〜J3 のパッド順（三角から 黒・赤・白・黄）を検査する。
  rev A のデータでは、J1〜J3 で失敗する
- 製造データ（ガーバー zip、ドリル、レンダリング、1:1 印刷用 PDF）を再生成
- 古い rev A の一式の zip（lte-power-switch.zip）を削除（注文データは git の履歴にある）
- README・docs を rev B の内容に更新

KiCad の DRC・ERC は違反 0 件。未発注。

Co-Authored-By: Claude Sonnet 5.5 <noreply@anthropic.com>
Parts:
- moved TP2 2.00 mm to (124.0, 88.0)
Routing:
- net /LTE_EN: track 8.20 -> 14.2 mm
- net /V3V3_IN: track 9.50 -> 11.1 mm
- net /VLTE: track 13.5 -> 14.2 mm
- net /SIG2: vias 4 -> 2
Other:
- board text added: "J1: GND 3V3 TX6(w) RX7(y)"
- board text added: "J2: GND VLTE RX(w) TX(y)"
- board text added: "J3 white=D1 shared w/ pot: keep NC"
- board text added: "J3: GND NC NC LTE_EN(y,D0)"
- board text added: "from triangle: black red white yellow"
- board text added: "rev B #88"
- board text added: "tri=GND(black)"
- board text removed: "1 yellow SIG1 2 white SIG2"
- board text removed: "3 red VCC 4 black GND"
- board text removed: "3V3"
- board text removed: "J1.3=3V3 in J2.3=VLTE out"
- board text removed: "J3: 1=LTE_EN 2,3=NC (no 5V)"
- board text removed: "rev A #88"
- board text removed: "triangle on top side = pin1"
